Commit message: add_gripper and scene

File: single_arm_description/config/single_arm_demo.urdf.xacro (robot description, xacro)
@@ -3,9 +3,19 @@
   <xacro:include filename="$(find single_arm_description)/urdf/single_arm.urdf.xacro" />
   <xacro:include filename="$(find single_arm_description)/config/single_arm.ros2_control.xacro" />
+  <xacro:include filename="$(find single_arm_description)/urdf/scene.urdf.xacro" />
+  <xacro:include filename="$(find single_arm_description)/urdf/gripper.urdf.xacro" />
+<!-- 在机械臂末端添加夹爪 -->
   <link name="world"/>
-  <xacro:single_arm name="single_arm_demo" parent="world">
-    <origin xyz="0 0 0" rpy="0 0 0"/>
+  <xacro:scene parent="world">
+    <!-- 可选整体偏移，如果想把平台放在某个位置 -->
+    <origin xyz="0 0 0.98" rpy="0 0 0"/>
+  </xacro:scene>
+  <xacro:single_arm name="single_arm" parent="optical_table">
+    <origin xyz="0 0 0.0" rpy="0 0 0"/>
   </xacro:single_arm>
+  <xacro:gripper name="gripper" parent="Empty_Link6">
+    <origin xyz="0 0 0.019" rpy="0 0 0"/>  <!-- 调整到合适姿态，通常和joint6的origin对齐 -->
+  </xacro:gripper>
   <xacro:single_arm_ros2_control
-    sim="false" namespace="" />
+    sim="true" namespace="" />
 </robot>

File: single_arm_description/urdf/single_arm.urdf.xacro (robot description, xacro)
@@ -40,5 +40,5 @@
         <geometry>
           <mesh
-            filename="package://single_arm_description/meshes/collision/base_link0.STL" />
+            filename="package://single_arm_description/meshes/collision/base_link0_simplified.STL" />
         </geometry>
       </collision>
@@ -87,5 +87,5 @@
         <geometry>
           <mesh
-            filename="package://single_arm_description/meshes/collision/Empty_Link1.STL" />
+            filename="package://single_arm_description/meshes/collision/Empty_Link1_simplified.STL" />
         </geometry>
       </collision>
@@ -145,5 +145,5 @@
         <geometry>
           <mesh
-            filename="package://single_arm_description/meshes/collision/Empty_Link2.STL" />
+            filename="package://single_arm_description/meshes/collision/Empty_Link2_simplified.STL" />
         </geometry>
       </collision>
@@ -203,5 +203,5 @@
         <geometry>
           <mesh
-            filename="package://single_arm_description/meshes/collision/Empty_Link3.STL" />
+            filename="package://single_arm_description/meshes/collision/Empty_Link3_simplified.STL" />
         </geometry>
       </collision>
@@ -319,5 +319,5 @@
         <geometry>
           <mesh
-            filename="package://single_arm_description/meshes/collision/Empty_Link5.STL" />
+            filename="package://single_arm_description/meshes/collision/Empty_Link5_simplified.STL" />
         </geometry>
       </collision>
@@ -378,5 +378,5 @@
         <geometry>
           <mesh
-            filename="package://single_arm_description/meshes/collision/Empty_Link6.STL" />
+            filename="package://single_arm_description/meshes/collision/Empty_Link6_simplified.STL" />
         </geometry>
       </collision>

Commit message: add obstacle

File: single_arm_description/config/single_arm_demo.urdf.xacro (robot description, xacro)
@@ -9,8 +9,8 @@
   <xacro:scene parent="world">
     <!-- 可选整体偏移，如果想把平台放在某个位置 -->
-    <origin xyz="0 0 0.98" rpy="0 0 0"/>
+    <origin xyz="0 0 0.8" rpy="0 0 0"/>
   </xacro:scene>
   <xacro:single_arm name="single_arm" parent="optical_table">
-    <origin xyz="0 0 0.0" rpy="0 0 0"/>
+    <origin xyz="-0.39 0.31 0.0" rpy="0 0 0"/>
   </xacro:single_arm>
   <xacro:gripper name="gripper" parent="Empty_Link6">

File: single_arm_description/urdf/scene.urdf.xacro (robot description, xacro)
@@ -29,4 +29,36 @@
       </inertial>
     </link>
+    <link name="obstacle_box">
+      <visual>
+        <!-- 底面放在平台表面（z=0），高度0.6m，中心抬高0.3m -->
+        <origin xyz="-0.78 0.11 0.6" rpy="0 0 1.5707963"/>
+        <geometry>
+          <box size="0.05 0.5 1.2"/>  <!-- x=0.4m, y=0.6m, z=0.6m，可自行调整 -->
+        </geometry>
+        <material name="obstacle_red">
+          <color rgba="0.8 0.2 0.2 1.0"/>  <!-- 红色，便于在RViz中识别 -->
+        </material>
+      </visual>
+      <collision>
+        <origin xyz="-0.78 0.11 0.6" rpy="0 0 1.5707963"/>
+        <geometry>
+          <box size="0.05 0.5 1.2"/>
+        </geometry>
+      </collision>
+      <!-- 可选惯性 -->
+      <inertial>
+        <origin xyz="-0.78 0.11 0.6" rpy="0 0 1.5707963"/>
+        <mass value="10.0"/>
+        <inertia ixx="1.0" ixy="0" ixz="0" iyy="1.0" iyz="0" izz="1.0"/>
+      </inertial>
+    </link>
+    <!-- 障碍物固定到world（与平台同层级） -->
+    <joint name="obstacle_box_joint" type="fixed">
+      <parent link="${parent}"/>
+      <child link="obstacle_box"/>
+      <!-- 位置：放在平台右边（x正方向偏移1.2m），y=0，底面z=0 -->
+      <!-- 你可以根据实际平台尺寸调整偏移量 -->
+      <origin xyz="0 0 0" rpy="0 0 0"/>
+    </joint>
     <!-- 把光学平台固定到world（或parent） -->
     <joint name="optical_table_joint" type="fixed">

Commit message: fix bugs

File: single_arm_description/config/single_arm_demo.urdf.xacro (robot description, xacro)
@@ -6,4 +6,6 @@
   <xacro:include filename="$(find single_arm_description)/urdf/gripper.urdf.xacro" />
 <!-- 在机械臂末端添加夹爪 -->
+  <xacro:arg name="sim" default="false" />
+  <xacro:arg name="use_gripper" default="true" />
   <link name="world"/>
   <xacro:scene parent="world">
@@ -14,8 +16,10 @@
     <origin xyz="-0.39 0.31 0.0" rpy="0 0 0"/>
   </xacro:single_arm>
-  <xacro:gripper name="gripper" parent="Empty_Link6">
-    <origin xyz="0 0 0.019" rpy="0 0 0"/>  <!-- 调整到合适姿态，通常和joint6的origin对齐 -->
-  </xacro:gripper>
+  <xacro:if value="$(arg use_gripper)">
+    <xacro:gripper name="gripper" parent="Empty_Link6">
+      <origin xyz="0 0 0.019" rpy="0 0 0"/>
+    </xacro:gripper>
+  </xacro:if>
   <xacro:single_arm_ros2_control
-    sim="true" namespace="" />
+    sim="$(arg sim)" namespace="" />
 </robot>

File: single_arm_description/urdf/scene.urdf.xacro (robot description, xacro)
@@ -29,13 +29,12 @@
       </inertial>
     </link>
-    <link name="obstacle_box">
+    <!-- <link name="obstacle_box">
       <visual>
-        <!-- 底面放在平台表面（z=0），高度0.6m，中心抬高0.3m -->
         <origin xyz="-0.78 0.11 0.6" rpy="0 0 1.5707963"/>
         <geometry>
-          <box size="0.05 0.5 1.2"/>  <!-- x=0.4m, y=0.6m, z=0.6m，可自行调整 -->
+          <box size="0.05 0.5 1.2"/>
         </geometry>
         <material name="obstacle_red">
-          <color rgba="0.8 0.2 0.2 1.0"/>  <!-- 红色，便于在RViz中识别 -->
+          <color rgba="0.8 0.2 0.2 1.0"/>
         </material>
       </visual>
@@ -46,5 +45,4 @@
         </geometry>
       </collision>
-      <!-- 可选惯性 -->
       <inertial>
         <origin xyz="-0.78 0.11 0.6" rpy="0 0 1.5707963"/>
@@ -52,14 +50,10 @@
         <inertia ixx="1.0" ixy="0" ixz="0" iyy="1.0" iyz="0" izz="1.0"/>
       </inertial>
-    </link>
-    <!-- 障碍物固定到world（与平台同层级） -->
-    <joint name="obstacle_box_joint" type="fixed">
+    </link> -->
+    <!-- <joint name="obstacle_box_joint" type="fixed">
       <parent link="${parent}"/>
       <child link="obstacle_box"/>
-      <!-- 位置：放在平台右边（x正方向偏移1.2m），y=0，底面z=0 -->
-      <!-- 你可以根据实际平台尺寸调整偏移量 -->
       <origin xyz="0 0 0" rpy="0 0 0"/>
-    </joint>
-    <!-- 把光学平台固定到world（或parent） -->
+    </joint> -->
     <joint name="optical_table_joint" type="fixed">
       <parent link="${parent}"/>

File: single_arm_description/urdf/single_arm.urdf.xacro (robot description, xacro)
@@ -160,5 +160,5 @@
         link="Empty_Link2" />
       <axis
-        xyz="0 0 1" />
+        xyz="0 0 -1" />
       <limit
         lower="-1.57"
@@ -276,8 +276,8 @@
         link="Empty_Link4" />
       <axis
-        xyz="0 0 1" />
-      <limit
-        lower="-2.61"
-        upper="0.69"
+        xyz="0 0 -1" />
+      <limit
+        lower="-0.69"
+        upper="2.61"
         effort="0"
         velocity="0" />
@@ -393,5 +393,5 @@
         link="Empty_Link6" />
       <axis
-        xyz="0 0 -1" />
+        xyz="0 0 1" />
       <limit
         lower="-3.14"

Commit message: change robot arm position on table

File: single_arm_description/config/single_arm_demo.urdf.xacro (robot description, xacro)
@@ -14,5 +14,5 @@
   </xacro:scene>
   <xacro:single_arm name="single_arm" parent="optical_table">
-    <origin xyz="-0.39 0.31 0.0" rpy="0 0 0"/>
+    <origin xyz="0.39 0.31 0.0" rpy="0 0 1.5707963"/>
   </xacro:single_arm>
   <xacro:if value="$(arg use_gripper)">
